File: hardware/lcd.kicad_sch (KiCad schematic)
At the start: 1 part

Commit message: * 3V8 Power design fixed * Footprints assigned * Bom exported * PCB filter module placed
Other:
- company: (none) -> Hidro Elektronik
- title: (none) -> 2023 Staj Projesi
Changed lines of the file:
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@@
 (kicad_sch (version 20230121) (generator eeschema)
   (paper "A4")
+  (title_block
+    (title "2023 Staj Projesi")
+    (date "2023-07-24")
+    (rev "1.0")
+    (company "Hidro Elektronik")
+    (comment 1 "Mehmet Emre SAYGI(2019513057@ogr.cu.edu.tr)")
+    (comment 2 "Yilmaz Can DURAN(duranyilmazcan@gmail.com)")
+    (comment 3 "Asli VEZIR(vezirasli@gmail.com)")
+  )
   (wire (pts (xy 144.78 80.01) (xy 154.94 80.01))
     (stroke (width 0) (type default))
@@
   (symbol (lib_id "power:+5V") (at 144.78 69.85 0) (unit 1)
     (in_bom yes) (on_board yes) (dnp no) (fields_autoplaced)
-    (property "Reference" "#PWR025" (at 144.78 73.66 0)
+    (property "Reference" "#PWR038" (at 144.78 73.66 0)
       (effects (font (size 1.27 1.27)) hide)
     )
@@
       (project "2023-staj-projesi"
         (path "/069db7ad-35cd-4aa8-8111-e026f632a4df/9df18327-ad01-4780-8291-2b0f280e8588"
-          (reference "#PWR025") (unit 1)
+          (reference "#PWR038") (unit 1)
         )
       )
@@
   (symbol (lib_id "power:GND") (at 148.59 93.98 0) (unit 1)
     (in_bom yes) (on_board yes) (dnp no) (fields_autoplaced)
-    (property "Reference" "#PWR024" (at 148.59 100.33 0)
+    (property "Reference" "#PWR039" (at 148.59 100.33 0)
       (effects (font (size 1.27 1.27)) hide)
     )
@@
       (project "2023-staj-projesi"
         (path "/069db7ad-35cd-4aa8-8111-e026f632a4df/9df18327-ad01-4780-8291-2b0f280e8588"
-          (reference "#PWR024") (unit 1)
+          (reference "#PWR039") (unit 1)
         )
       )
